File: KiCad/AlarmClock.kicad_sch (KiCad schematic)
At the start: 75 parts, among them SW1 RotaryEncoder_Switch, SW2 SW_SPST, SW3 SW_Push, U1 D168K, U10 TPIC6595, U11 TPIC6595, U12 TPIC6595, U13 TPIC6595, U14 TPIC6595, U15 TPIC6595, U2 D168K, U3 D168K, U4 D168K, U5 D168K, U6 D168K, U7 RC1602A, U8 TPIC6595, U9 TPIC6595

Commit message: reformat your questionable schematic, and import components into pcb editor
Parts:
- R1, R10, R11, R12, R13, R14, R15, R16, R17, R18, R19, R2, R20, R21, R22, R23, R24, R25, R26, R27, R28, R29, R3, R30, R31, R32, R33, R34, R35, R36, R37, R38, R39, R4, R40, R41, R42, R43, R44, R45, R46, R47, R48, R49, R5, R6, R7, R8, R9: footprint (none) -> Resistor_SMD:R_0402_1005Metric
- SW3: footprint ScottoKeebs_MX:MX_PCB_1.00u -> PCM_marbastlib-mx:SW_MX_1u
Connections:
- net Char LCD SR CLK: now also U14.13 (SRCK); no longer U14.3 (SER_IN)
- net Char LCD SR SI: now also U14.3 (SER_IN); no longer U14.13 (SRCK)
- net LED SR SI: no longer U15.3 (SER_IN)
- net Snooze button: now also U15.3 (SER_IN)
- no-connect marks 45 -> 46
Other:
- note added: "Buzzer"
- note added: "Delimiters & Buttons"
- note added: "Rotary Encoder"
- note added: "Segmented Displays"
- note added: "Socketed Arduino"
- moved on the sheet: A1, BZ1, D10, D5, D6, D7, D8, D9, R1, R10, R18, R2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
